Commit message: OK_1

File: src/hospital_robot/urdf/omni_base.urdf (robot description, URDF)
Before this commit: robot omni_base, 17 links, 16 joints
Links:
- added link camera_link, mass 0.1; collision box size=0.05 0.05 0.05; visual box size=0.05 0.05 0.05
Joints:
- added joint camera_joint: type fixed, parent base_link, child camera_link, origin xyz=0.35 0 0.3 rpy=0 0 0
